File: stm32f030_dev_board.kicad_sch (KiCad schematic)
At the start: 62 parts, among them J2 Conn_01x16, J3 Conn_01x16, J4 Conn_01x16, J5 Conn_01x06, J6 Conn_01x04, J7 USB_C_Receptacle_USB2.0_16P, Q1 DMP3099L, Q2 DMP3099L, SW1 SW_Push, SW3 SW_Push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

Commit message: Started PCB layout and added net labels to schematic
Parts:
- removed Y3: 32.768KHz, Crystal:Crystal_SMD_Abracon_ABS25-4Pin_8.0x3.8mm, symbol Device:Crystal
- added Y3: 32.768kHz, Crystal:Crystal_SMD_Abracon_ABS25-4Pin_8.0x3.8mm, symbol Device:Crystal_GND23
- Y2: footprint Crystal:Crystal_HC49-U_Vertical -> Crystal:Crystal_HC49-4H_Vertical
Connections:
- net GND: now also Y3.2, Y3.3
- net OSC32_IN: now also Y3.1
- net OSC32_OUT: now also Y3.4
- net OSC_OUT_R: now reaches C24.1, R10.2, Y2.1
- net XCSI: now reaches C21.1, U2.1 (XCSI), Y1.1
- net XCSO: now reaches C22.1, U2.2 (XCSO), Y1.2
- net VCCA: now reaches C12.2, U2.37 (VCCA)
- net BOOT0: now reaches R9.1, U1.60 (BOOT0)
- net SW_R: now reaches R9.2, S1.2
- net RESET: now reaches R8.1, U2.34 (~{RESET})
- net VCCCORE: now reaches C13.2, U2.38 (VCCCORE)
- net REF: now reaches R7.1, U2.5 (REF)
- net DM: now reaches R5.1, U2.6 (DM)
- net DP: now reaches R6.1, U2.7 (DP)
Other:
- moved on the sheet: C12, C13, C26

Commit message: Layout the pcb and added mounting holes to schematic and pcb
Parts:
- added H1, H2, H3, H4: MountingHole, MountingHole:MountingHole_2.2mm_M2, symbol Mechanical:MountingHole
Connections:
- net VI: now reaches C28.1, Q1.2 (S), Q2.2 (S), U3.3 (VI)
- net CC1: now reaches J7.A5 (CC1), R3.1
- net CC2: now reaches J7.B5 (CC2), R4.2
- net LED+: now reaches D1.2 (A), R13.1
Other:
- note added: "M3"
- note added: "Mounting Holes"
- moved on the sheet: R3, R4

Commit message: removed D+ and D- resistors, finished routing front and back copper, moved button to better place
Parts:
- removed R5, R6: 22, Resistor_SMD:R_0603_1608Metric_Pad0.98x0.95mm_HandSolder, symbol Device:R
Connections:
- net DM is gone; now on net D-: U2.6 (DM)
- net DP is gone; now on net D+: U2.7 (DP)
- net GND: now also J4.15 (Pin_15)
- no-connect marks 22 -> 21
Changed lines of the file:
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@@
 	)
 	(no_connect
-		(at 53.34 52.07)
-	)
-	(no_connect
 		(at 182.88 57.15)
 	)
@@
 	(wire
 		(pts
-			(xy 222.25 46.99) (xy 227.33 46.99)
-		)
-		(stroke
-			(width 0)
-			(type default)
-		)
-	)
-	(wire
-		(pts
 			(xy 69.85 58.42) (xy 69.85 62.23)
 		)
@@
 	(wire
 		(pts
+			(xy 49.53 52.07) (xy 53.34 52.07)
+		)
+		(stroke
+			(width 0)
+			(type default)
+		)
+	)
+	(wire
+		(pts
 			(xy 21.59 160.02) (xy 21.59 161.29)
 		)
@@
 	(wire
 		(pts
-			(xy 210.82 44.45) (xy 214.63 44.45)
-		)
-		(stroke
-			(width 0)
-			(type default)
-		)
-	)
-	(wire
-		(pts
 			(xy 223.52 129.54) (xy 223.52 130.81)
 		)
@@
 	(wire
 		(pts
+			(xy 220.98 46.99) (xy 227.33 46.99)
+		)
+		(stroke
+			(width 0)
+			(type default)
+		)
+	)
+	(wire
+		(pts
 			(xy 71.12 173.99) (xy 64.77 173.99)
 		)
@@
 	(wire
 		(pts
+			(xy 220.98 44.45) (xy 227.33 44.45)
+		)
+		(stroke
+			(width 0)
+			(type default)
+		)
+	)
+	(wire
+		(pts
 			(xy 255.27 20.32) (xy 252.73 20.32)
 		)
@@
 	(wire
 		(pts
-			(xy 210.82 46.99) (xy 214.63 46.99)
-		)
-		(stroke
-			(width 0)
-			(type default)
-		)
-	)
-	(wire
-		(pts
 			(xy 255.27 21.59) (xy 255.27 20.32)
 		)
@@
 	(wire
 		(pts
-			(xy 222.25 44.45) (xy 227.33 44.45)
-		)
-		(stroke
-			(width 0)
-			(type default)
-		)
-	)
-	(wire
-		(pts
 			(xy 30.48 115.57) (xy 30.48 116.84)
 		)
@@
 	)
 	(label "D-"
-		(at 210.82 44.45 0)
+		(at 220.98 44.45 0)
 		(effects
 			(font
@@
 	)
 	(label "D+"
-		(at 210.82 46.99 0)
+		(at 220.98 46.99 0)
 		(effects
 			(font
@@
 		)
 	)
-	(label "DP"
-		(at 223.52 46.99 0)
-		(effects
-			(font
-				(size 1.27 1.27)
-			)
-			(justify left bottom)
-		)
-	)
 	(label "PA5"
 		(at 93.98 82.55 0)
@@
 		)
 	)
-	(label "DM"
-		(at 223.52 44.45 0)
-		(effects
-			(font
-				(size 1.27 1.27)
-			)
-			(justify left bottom)
-		)
-	)
 	(label "PC6"
 		(at 53.34 31.75 180)
@@
 	)
 	(symbol
-		(lib_id "Device:R")
-		(at 218.44 46.99 270)
-		(unit 1)
-		(exclude_from_sim no)
-		(in_bom yes)
-		(on_board yes)
-		(dnp no)
-		(property "Reference" "R6"
-			(at 218.44 49.276 90)
-			(effects
-				(font
-					(size 1.27 1.27)
-				)
-			)
-		)
-		(property "Value" "22"
-			(at 218.44 46.99 90)
-			(effects
-				(font
-					(size 1.27 1.27)
-				)
-			)
-		)
-		(property "Footprint" "Resistor_SMD:R_0603_1608Metric_Pad0.98x0.95mm_HandSolder"
-			(at 218.44 45.212 90)
-			(effects
-				(font
-					(size 1.27 1.27)
-				)
-				(hide yes)
-			)
-		)
-		(property "Datasheet" "~"
-			(at 218.44 46.99 0)
-			(effects
-				(font
-					(size 1.27 1.27)
-				)
-				(hide yes)
-			)
-		)
-		(property "Description" "Resistor"
-			(at 218.44 46.99 0)
-			(effects
-				(font
-					(size 1.27 1.27)
-				)
-				(hide yes)
-			)
-		)
-		(pin "2"
-		)
-		(pin "1"
-		)
-		(instances
-			(project "stm32f030"
-				(path "/c745f8ec-5d7c-4e57-8ba7-8ae1e0dd3053"
-					(reference "R6")
-					(unit 1)
-				)
-			)
-		)
-	)
-	(symbol
 		(lib_id "Device:C")
 		(at 276.86 123.19 0)
@@
 	)
 	(symbol
+		(lib_id "power:GND")
+		(at 49.53 52.07 270)
+		(unit 1)
+		(exclude_from_sim no)
+		(in_bom yes)
+		(on_board yes)
+		(dnp no)
+		(fields_autoplaced yes)
+		(property "Reference" "#PWR02"
+			(at 43.18 52.07 0)
+			(effects
+				(font
+					(size 1.27 1.27)
+				)
+				(hide yes)
+			)
+		)
+		(property "Value" "GND"
+			(at 45.72 52.0699 90)
+			(effects
+				(font
+					(size 1.27 1.27)
+				)
+				(justify right)
+			)
+		)
+		(property "Footprint" ""
+			(at 49.53 52.07 0)
+			(effects
+				(font
+					(size 1.27 1.27)
+				)
+				(hide yes)
+			)
+		)
+		(property "Datasheet" ""
+			(at 49.53 52.07 0)
+			(effects
+				(font
+					(size 1.27 1.27)
+				)
+				(hide yes)
+			)
+		)
+		(property "Description" "Power symbol creates a global label with name \"GND\" , ground"
+			(at 49.53 52.07 0)
+			(effects
+				(font
+					(size 1.27 1.27)
+				)
+				(hide yes)
+			)
+		)
+		(pin "1"
+		)
+		(instances
+			(project ""
+				(path "/c745f8ec-5d7c-4e57-8ba7-8ae1e0dd3053"
+					(reference "#PWR02")
+					(unit 1)
+				)
+			)
+		)
+	)
+	(symbol
 		(lib_id "power:PWR_FLAG")
 		(at 29.21 69.85 0)
@@
 					(unit 1)
 				)
-			)
-		)
-	)
-	(symbol
-		(lib_id "Device:R")
-		(at 218.44 44.45 270)
-		(unit 1)
-		(exclude_from_sim no)
-		(in_bom yes)
-		(on_board yes)
-		(dnp no)
-		(property "Reference" "R5"
-			(at 218.44 42.418 90)
-			(effects
-				(font
-					(size 1.27 1.27)
-				)
-			)
-		)
-		(property "Value" "22"
-			(at 218.694 44.45 90)
-			(effects
-				(font
-					(size 1.27 1.27)
-				)
-			)
-		)
-		(property "Footprint" "Resistor_SMD:R_0603_1608Metric_Pad0.98x0.95mm_HandSolder"
-			(at 218.44 42.672 90)
-			(effects
-				(font
-					(size 1.27 1.27)
-				)
-				(hide yes)
-			)
-		)
-		(property "Datasheet" "~"
-			(at 218.44 44.45 0)
-			(effects
-				(font
-					(size 1.27 1.27)
-				)
-				(hide yes)
-			)
-		)
-		(property "Description" "Resistor"
-			(at 218.44 44.45 0)
-			(effects
-				(font
-					(size 1.27 1.27)
-				)
-				(hide yes)
-			)
-		)
-		(pin "2"
-		)
-		(pin "1"
-		)
-		(instances
-			(project "stm32f030"
-				(path "/c745f8ec-5d7c-4e57-8ba7-8ae1e0dd3053"
-					(reference "R5")
-					(unit 1)
-				)
